File: rev.1/rev.1.kicad_sch (KiCad schematic)
At the start: 129 parts, among them Q1 BC857, Q2 BC817, SW1 RESET, SW2 POWER, X1 POWER, X2 Манипулятор_1, X3 AUDIO_1, X4 AUDIO_2, X5 Манипулятор_2, X6 VIDEO

Commit message: Сделал разводку печатной платы
Parts:
- removed D4: SS14, Diode_SMD:D_SMA, symbol Diode_Schottky_gost:SS14
- added C10, C2: 0.1uF, Capacitor_SMD:C_0603_1608Metric, symbol Device:C_Small
- added D4: BAS85, Diode_SMD:D_MiniMELF, symbol Diode_Schottky_gost:BAS85
- C23: renamed from C21; footprint Capacitor_THT:CP_Radial_D6.3mm_P2.50mm -> Capacitor_SMD:CP_Elec_4x5.4
- C24: renamed from C22; footprint Capacitor_THT:CP_Radial_D6.3mm_P2.50mm -> Capacitor_SMD:CP_Elec_4x5.4
- C28: renamed from C26; footprint Capacitor_THT:CP_Radial_D6.3mm_P2.50mm -> Capacitor_SMD:CP_Elec_4x5.4
- C3: renamed from C2; footprint Capacitor_THT:CP_Radial_D10.0mm_P5.00mm -> Capacitor_SMD:CP_Elec_8x10.5
- C36: renamed from C34; footprint Capacitor_THT:CP_Radial_D6.3mm_P2.50mm -> Capacitor_SMD:CP_Elec_4x5.4
- C37: renamed from C35; footprint Capacitor_THT:CP_Radial_D6.3mm_P2.50mm -> Capacitor_SMD:CP_Elec_4x5.4
- C41: renamed from C39; footprint Capacitor_THT:CP_Radial_D7.5mm_P2.50mm -> Capacitor_SMD:CP_Elec_8x6.5
- C9: renamed from C8; footprint Capacitor_THT:CP_Radial_D6.3mm_P2.50mm -> Capacitor_SMD:CP_Elec_8x10.5
- SW1: footprint Button_Switch_THT:SW_PUSH_6mm_H7.3mm -> Button_Switch_THT:KLS7_P8X8; symbol Switch:SW_Push_Dual -> Switch:SW_Push_6
- SW2: footprint Button_Switch_THT:Nidec_Copal_SH-7010C -> Button_Switch_THT:KLS7_P8X8; symbol Switch:SW_Push_Dual -> Switch:SW_Push_6
- X3, X4, X6: footprint Connector_Audio:rca_red -> Connector_Audio:RCA-105; symbol Connectors_gost:Conn_01x04_Female -> Connectors_gost:Conn_01x03_Female
- renumbered C9 to C11, C10 to C12, C11 to C13, C12 to C14, C13 to C15, C14 to C16, C15 to C17, C16 to C18, C17 to C19, C18 to C20, C19 to C21, C20 to C22, C23 to C25, C24 to C26, C25 to C27, C27 to C29, C28 to C30, C29 to C31, C30 to C32, C31 to C33, C32 to C34, C33 to C35, C36 to C38, C37 to C39, C3 to C4, C38 to C40, C40 to C42, C41 to C43, C42 to C44, C4 to C5, C5 to C6, C6 to C7, C7 to C8
Connections:
- net +5V: now also C10.1
- net GNDD: now also SW1.2, C10.2, C2.2; no longer SW1.1, X3.4 (Pin_4), X4.4 (Pin_4), X6.4 (Pin_4)
- net RESET: now also SW1.5; no longer SW1.2
- net at D1.1 (K), SW2.3: now also SW2.2; no longer SW2.1
- net at Q2.1 (B), R31.1, R32.2: now also D4.1 (K)
- net at C41.1, Q2.2 (E), R41.2: now also D4.2 (A)
- net at C3.1, DA1.6 (Vin), R3.1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: now also SW2.5, C2.1; no longer SW2.2
Other:
- moved on the sheet: R3

Commit message: добавил список элементов ,гербера
Parts:
- C1: MNF# (none) -> CC0603KRX7R9BB474
- C10, C11, C12, C13, C14, C15, C16, C17, C18, C19, C2, C22, C25, C26, C27, C4, C42, C43, C44, C5, C6, C8: MNF# (none) -> CC0603ZRY5V9BB104
- C20, C21, C29, C32, C33, C34, C35, C38, C39, C40: MNF# (none) -> CC0603JRNPO9BN331
- C23, C24, C28, C36, C37: MNF# (none) -> CK1C100M-CRC54
- C3: MNF# (none) -> VT221M1EJBKJ0810VBK
- C30, C31: MNF# (none) -> CC0603JRNPO9BN220
- C41: MNF# (none) -> VCT227M010S0ANG10L
- C7: MNF# (none) -> CC0603KRX7R9BB471
- C9: MNF# (none) -> TS13C00J471MJT000R
- D1, D2: MNF# (none) -> SS14
- D3: value POWER -> LED_POWER; MNF# (none) -> L-7104EC@KGB
- D4: MNF# (none) -> BAS85
- DA1: MNF# (none) -> MC34063AD
- DA2: MNF# (none) -> LM358D
- DD1: MNF# (none) -> UA6527P
- DD2: MNF# (none) -> UA6538
- DD3: MNF# (none) -> 74HC373D
- DD4: MNF# (none) -> 74HC139D
- DD5, DD6: MNF# (none) -> IS62C256AL-45ULI
- DD7, DD8: MNF# (none) -> 74HC368D
- DD9: MNF# (none) -> SN74LS04D
- L1, L10, L11, L12, L13, L14, L15, L16, L2, L3, L5, L6, L7, L8, L9: MNF# (none) -> BLM18EG221SN1D
- L4: MNF# (none) -> RLB0914-221KL
- Q1: MNF# (none) -> BC857B
- Q2: MNF# (none) -> BC817-25
- R1, R11, R2, R27, R28, R29, R30, R33, R36, R38, R39, R40, R42, R44, R7, R8: MNF# (none) -> RC0603FR-0710KL
- R10, R43, R9: MNF# (none) -> RC0603FR-0775RL
- R12, R31: MNF# (none) -> RC0603FR-072K2L
- R13, R17: MNF# (none) -> RC0603FR-072KL
- R14, R25, R26: MNF# (none) -> RC0603FR-071KL
- R15, R18, R19, R20, R21, R22: MNF# (none) -> RC0603FR-074K7L
- R16: MNF# (none) -> RC0603FR-071K8L
- R23, R24: MNF# (none) -> RC0603FR-07510RL
- R3: MNF# (none) -> RL0603FR-070R1L
- R32: MNF# (none) -> RC0603FR-07220RL
- R34, R35: MNF# (none) -> RC0603FR-071RL
- R37: MNF# (none) -> RC0603FR-074M7L
- R4: MNF# (none) -> RC0603FR-073K6L
- R41: MNF# (none) -> RC0603FR-0768RL
- R5: MNF# (none) -> RC0603FR-071K2L
- R6: MNF# (none) -> RC0603FR-07330RL
- SW1: MNF# (none) -> KLS7-P8.0*8.0-0
- SW2: value POWER -> BUT_POWER; MNF# (none) -> KLS7-P8.0*8.0-1
- X1: MNF# (none) -> KLS1-DC-005A-2.0
- X2, X5: MNF# (none) -> DS1037-15-MNAKT74-0CC
- X3, X4, X6: MNF# (none) -> RCA-103P
- XP1: MNF# (none) -> KLS1-603C-62-S
- Z1: MNF# (none) -> 26.601712M 20PF 30PPM
Connections:
- no-connect marks 16 -> 20
Other:
- company: (none) -> hamradio@conference.jabber.ru
- title: (none) -> Игровая приставка(клон famicom)
